Commit message: Pre-Simple Movement

File: src/jamie_description/urdf/jamie.xacro (robot description, xacro)
@@ -6,5 +6,5 @@
 <link name="base_link">
   <inertial>
-    <origin xyz="3.1106206943576354e-10 -0.001705459809340095 0.41858451888973675" rpy="0 0 0"/>
+    <origin xyz="-0.011688232223622823 -0.04997378243790669 -0.12088695327313781" rpy="0 0 0"/>
     <mass value="0.8307183918921939"/>
     <inertia ixx="0.000743" iyy="0.00316" izz="0.00283" ixy="0.0" iyz="3.2e-05" ixz="-0.0"/>
@@ -26,10 +26,10 @@
 <link name="right_shoulder_link_1">
   <inertial>
-    <origin xyz="0.0006456837649729541 0.02009213962856949 -0.018618587576526346" rpy="0 0 0"/>
+    <origin xyz="0.0006454512302885018 0.020091817000003336 -0.018619059739400937" rpy="0 0 0"/>
     <mass value="0.18884280500199657"/>
     <inertia ixx="7.8e-05" iyy="7.4e-05" izz="5.8e-05" ixy="-0.0" iyz="6e-06" ixz="1e-06"/>
   </inertial>
   <visual>
-    <origin xyz="-0.108676 0.005103 -0.673203" rpy="0 0 0"/>
+    <origin xyz="-0.096988 0.053371 -0.133732" rpy="0 0 0"/>
     <geometry>
       <mesh filename="package://jamie_description/meshes/right_shoulder_link_1.stl" scale="0.001 0.001 0.001"/>
@@ -38,5 +38,5 @@
   </visual>
   <collision>
-    <origin xyz="-0.108676 0.005103 -0.673203" rpy="0 0 0"/>
+    <origin xyz="-0.096988 0.053371 -0.133732" rpy="0 0 0"/>
     <geometry>
       <mesh filename="package://jamie_description/meshes/right_shoulder_link_1.stl" scale="0.001 0.001 0.001"/>
@@ -46,10 +46,10 @@
 <link name="left_shoulder_link_1">
   <inertial>
-    <origin xyz="-0.0006454231580610287 0.01898370677952162 -0.0197473856344742" rpy="0 0 0"/>
+    <origin xyz="-0.0006456556927465912 0.018983384150954692 -0.019747857797348778" rpy="0 0 0"/>
     <mass value="0.1888429783699795"/>
     <inertia ixx="7.8e-05" iyy="7.5e-05" izz="5.8e-05" ixy="0.0" iyz="5e-06" ixz="-1e-06"/>
   </inertial>
   <visual>
-    <origin xyz="0.106476 0.004911 -0.673264" rpy="0 0 0"/>
+    <origin xyz="0.118164 0.053179 -0.133793" rpy="0 0 0"/>
     <geometry>
       <mesh filename="package://jamie_description/meshes/left_shoulder_link_1.stl" scale="0.001 0.001 0.001"/>
@@ -58,5 +58,5 @@
   </visual>
   <collision>
-    <origin xyz="0.106476 0.004911 -0.673264" rpy="0 0 0"/>
+    <origin xyz="0.118164 0.053179 -0.133793" rpy="0 0 0"/>
     <geometry>
       <mesh filename="package://jamie_description/meshes/left_shoulder_link_1.stl" scale="0.001 0.001 0.001"/>
@@ -66,10 +66,10 @@
 <link name="chest_link_1">
   <inertial>
-    <origin xyz="1.1937011133657423e-07 0.02906262980492068 0.04593037735780203" rpy="0 0 0"/>
+    <origin xyz="-1.1316457350710185e-07 0.02906330717635416 0.04592990519492751" rpy="0 0 0"/>
     <mass value="1.8523759675731215"/>
     <inertia ixx="0.001182" iyy="0.003891" izz="0.004278" ixy="-0.0" iyz="5.8e-05" ixz="-0.0"/>
   </inertial>
   <visual>
-    <origin xyz="-0.0011 0.009084 -0.623779" rpy="0 0 0"/>
+    <origin xyz="0.010588 0.057353 -0.084308" rpy="0 0 0"/>
     <geometry>
       <mesh filename="package://jamie_description/meshes/chest_link_1.stl" scale="0.001 0.001 0.001"/>
@@ -78,5 +78,5 @@
   </visual>
   <collision>
-    <origin xyz="-0.0011 0.009084 -0.623779" rpy="0 0 0"/>
+    <origin xyz="0.010588 0.057353 -0.084308" rpy="0 0 0"/>
     <geometry>
       <mesh filename="package://jamie_description/meshes/chest_link_1.stl" scale="0.001 0.001 0.001"/>
@@ -86,10 +86,10 @@
 <link name="spine_connector_link_1">
   <inertial>
-    <origin xyz="-0.016505894109137692 0.009764624496856791 0.010210578077430865" rpy="0 0 0"/>
+    <origin xyz="-0.016506126643822533 0.00976530186829027 0.010210105914556483" rpy="0 0 0"/>
     <mass value="0.2675520479560331"/>
     <inertia ixx="0.000166" iyy="0.000125" izz="0.000109" ixy="1.4e-05" iyz="-1e-06" ixz="1e-06"/>
   </inertial>
   <visual>
-    <origin xyz="-0.0236 -0.005166 -0.623779" rpy="0 0 0"/>
+    <origin xyz="-0.011912 0.043103 -0.084308" rpy="0 0 0"/>
     <geometry>
       <mesh filename="package://jamie_description/meshes/spine_connector_link_1.stl" scale="0.001 0.001 0.001"/>
@@ -98,5 +98,5 @@
   </visual>
   <collision>
-    <origin xyz="-0.0236 -0.005166 -0.623779" rpy="0 0 0"/>
+    <origin xyz="-0.011912 0.043103 -0.084308" rpy="0 0 0"/>
     <geometry>
       <mesh filename="package://jamie_description/meshes/spine_connector_link_1.stl" scale="0.001 0.001 0.001"/>
@@ -106,10 +106,10 @@
 <link name="left_upper_leg_link_1">
   <inertial>
-    <origin xyz="-0.01184936032213374 0.002829694297358378 -0.08923111810416501" rpy="0 0 0"/>
+    <origin xyz="-0.011849592856818726 0.002829371668791672 -0.08923059026703958" rpy="0 0 0"/>
     <mass value="0.40754083950250325"/>
     <inertia ixx="0.001416" iyy="0.001457" izz="0.000338" ixy="-1.7e-05" iyz="9e-05" ixz="0.00022"/>
   </inertial>
   <visual>
-    <origin xyz="0.0433 -0.014351 -0.394608" rpy="0 0 0"/>
+    <origin xyz="0.054988 0.033917 0.144864" rpy="0 0 0"/>
     <geometry>
       <mesh filename="package://jamie_description/meshes/left_upper_leg_link_1.stl" scale="0.001 0.001 0.001"/>
@@ -118,5 +118,5 @@
   </visual>
   <collision>
-    <origin xyz="0.0433 -0.014351 -0.394608" rpy="0 0 0"/>
+    <origin xyz="0.054988 0.033917 0.144864" rpy="0 0 0"/>
     <geometry>
       <mesh filename="package://jamie_description/meshes/left_upper_leg_link_1.stl" scale="0.001 0.001 0.001"/>
@@ -126,10 +126,10 @@
 <link name="right_upper_leg_link_1">
   <inertial>
-    <origin xyz="0.011850015567623058 0.0028296942840022182 -0.08923111810698131" rpy="0 0 0"/>
+    <origin xyz="0.011849783032938543 0.002829371655435887 -0.08923059026985594" rpy="0 0 0"/>
     <mass value="0.40754083973100536"/>
     <inertia ixx="0.001416" iyy="0.001457" izz="0.000338" ixy="1.7e-05" iyz="9e-05" ixz="-0.00022"/>
   </inertial>
   <visual>
-    <origin xyz="-0.0433 -0.014351 -0.394608" rpy="0 0 0"/>
+    <origin xyz="-0.031612 0.033917 0.144864" rpy="0 0 0"/>
     <geometry>
       <mesh filename="package://jamie_description/meshes/right_upper_leg_link_1.stl" scale="0.001 0.001 0.001"/>
@@ -138,5 +138,5 @@
   </visual>
   <collision>
-    <origin xyz="-0.0433 -0.014351 -0.394608" rpy="0 0 0"/>
+    <origin xyz="-0.031612 0.033917 0.144864" rpy="0 0 0"/>
     <geometry>
       <mesh filename="package://jamie_description/meshes/right_upper_leg_link_1.stl" scale="0.001 0.001 0.001"/>
@@ -146,10 +146,10 @@
 <link name="spine_link_1">
   <inertial>
-    <origin xyz="0.027174999999975347 0.0030514827161806863 0.08500010628608651" rpy="0 0 0"/>
+    <origin xyz="0.027174767465290472 0.0030521600876141017 0.08499963412321193" rpy="0 0 0"/>
     <mass value="0.2851299685332731"/>
     <inertia ixx="0.00083" iyy="0.00095" izz="0.000199" ixy="0.0" iyz="0.0" ixz="-0.0"/>
   </inertial>
   <visual>
-    <origin xyz="0.02725 -0.005166 -0.453779" rpy="0 0 0"/>
+    <origin xyz="0.038938 0.043103 0.085692" rpy="0 0 0"/>
     <geometry>
       <mesh filename="package://jamie_description/meshes/spine_link_1.stl" scale="0.001 0.001 0.001"/>
@@ -158,5 +158,5 @@
   </visual>
   <collision>
-    <origin xyz="0.02725 -0.005166 -0.453779" rpy="0 0 0"/>
+    <origin xyz="0.038938 0.043103 0.085692" rpy="0 0 0"/>
     <geometry>
       <mesh filename="package://jamie_description/meshes/spine_link_1.stl" scale="0.001 0.001 0.001"/>
@@ -166,10 +166,10 @@
 <link name="neck_servo_v1_1">
   <inertial>
-    <origin xyz="0.004498988710398971 -0.02468095859865068 -0.008128190094231602" rpy="0 0 0"/>
+    <origin xyz="0.004498756175713993 -0.024681281227217043 -0.00812866225710629" rpy="0 0 0"/>
     <mass value="0.25721902111029343"/>
     <inertia ixx="7.2e-05" iyy="4.5e-05" izz="4.3e-05" ixy="0.0" iyz="2e-06" ixz="0.0"/>
   </inertial>
   <visual>
-    <origin xyz="0.0034 -0.039771 -0.697879" rpy="0 0 0"/>
+    <origin xyz="0.015088 0.008497 -0.158408" rpy="0 0 0"/>
     <geometry>
       <mesh filename="package://jamie_description/meshes/neck_servo_v1_1.stl" scale="0.001 0.001 0.001"/>
@@ -178,5 +178,5 @@
   </visual>
   <collision>
-    <origin xyz="0.0034 -0.039771 -0.697879" rpy="0 0 0"/>
+    <origin xyz="0.015088 0.008497 -0.158408" rpy="0 0 0"/>
     <geometry>
       <mesh filename="package://jamie_description/meshes/neck_servo_v1_1.stl" scale="0.001 0.001 0.001"/>
@@ -186,10 +186,10 @@
 <link name="neck_link_1">
   <inertial>
-    <origin xyz="7.139401547438936e-06 0.008823511285371906 0.007600475444214827" rpy="0 0 0"/>
+    <origin xyz="7.906866862536846e-06 0.008823188656805377 0.007600003281340223" rpy="0 0 0"/>
     <mass value="0.09691779368254524"/>
     <inertia ixx="2.3e-05" iyy="5.3e-05" izz="5.3e-05" ixy="0.0" iyz="-1e-06" ixz="-0.0"/>
   </inertial>
   <visual>
-    <origin xyz="-0.001102 -0.005338 -0.713679" rpy="0 0 0"/>
+    <origin xyz="0.010587 0.04293 -0.174208" rpy="0 0 0"/>
     <geometry>
       <mesh filename="package://jamie_description/meshes/neck_link_1.stl" scale="0.001 0.001 0.001"/>
@@ -198,5 +198,5 @@
   </visual>
   <collision>
-    <origin xyz="-0.001102 -0.005338 -0.713679" rpy="0 0 0"/>
+    <origin xyz="0.010587 0.04293 -0.174208" rpy="0 0 0"/>
     <geometry>
       <mesh filename="package://jamie_description/meshes/neck_link_1.stl" scale="0.001 0.001 0.001"/>
@@ -206,10 +206,10 @@
 <link name="neck_nod_tilt_link_1">
   <inertial>
-    <origin xyz="0.016877140142823113 -0.009828122182642944 0.010518297464361615" rpy="0 0 0"/>
+    <origin xyz="0.016876907608138172 -0.009827444811209469 0.010517825301487094" rpy="0 0 0"/>
     <mass value="0.2884047672762395"/>
     <inertia ixx="0.000176" iyy="0.000137" izz="0.000111" ixy="1.6e-05" iyz="-5e-06" ixz="1e-06"/>
   </inertial>
   <visual>
-    <origin xyz="0.021885 -0.021358 -0.738679" rpy="0 0 0"/>
+    <origin xyz="0.033573 0.026911 -0.199208" rpy="0 0 0"/>
     <geometry>
       <mesh filename="package://jamie_description/meshes/neck_nod_tilt_link_1.stl" scale="0.001 0.001 0.001"/>
@@ -218,5 +218,5 @@
   </visual>
   <collision>
-    <origin xyz="0.021885 -0.021358 -0.738679" rpy="0 0 0"/>
+    <origin xyz="0.033573 0.026911 -0.199208" rpy="0 0 0"/>
     <geometry>
       <mesh filename="package://jamie_description/meshes/neck_nod_tilt_link_1.stl" scale="0.001 0.001 0.001"/>
@@ -226,10 +226,10 @@
 <link name="eye_holder_link_1">
   <inertial>
-    <origin xyz="5.980346964292956e-06 0.006609529389791653 1.0628523761102571e-07" rpy="0 0 0"/>
+    <origin xyz="5.747812279516609e-06 0.006610206761225312 -3.658776367987393e-07" rpy="0 0 0"/>
     <mass value="0.16148324488991492"/>
     <inertia ixx="6.3e-05" iyy="0.000324" izz="0.000261" ixy="0.0" iyz="-0.0" ixz="5e-06"/>
   </inertial>
   <visual>
-    <origin xyz="-0.000633 -0.042443 -0.782179" rpy="0 0 0"/>
+    <origin xyz="0.011055 0.005826 -0.242708" rpy="0 0 0"/>
     <geometry>
       <mesh filename="package://jamie_description/meshes/eye_holder_link_1.stl" scale="0.001 0.001 0.001"/>
@@ -238,5 +238,5 @@
   </visual>
   <collision>
-    <origin xyz="-0.000633 -0.042443 -0.782179" rpy="0 0 0"/>
+    <origin xyz="0.011055 0.005826 -0.242708" rpy="0 0 0"/>
     <geometry>
       <mesh filename="package://jamie_description/meshes/eye_holder_link_1.stl" scale="0.001 0.001 0.001"/>
@@ -246,10 +246,10 @@
 <link name="head_connector_link_1">
   <inertial>
-    <origin xyz="-1.995390094584621e-05 -0.023605835187592815 0.020398942883291915" rpy="0 0 0"/>
+    <origin xyz="-2.018643563084059e-05 -0.023606157816159382 0.0203984707204177" rpy="0 0 0"/>
     <mass value="0.10736239781961848"/>
     <inertia ixx="0.000111" iyy="2e-05" izz="0.000103" ixy="-0.0" iyz="-2e-06" ixz="-0.0"/>
   </inertial>
   <visual>
-    <origin xyz="-0.000627 -0.035338 -0.759679" rpy="0 0 0"/>
+    <origin xyz="0.011061 0.01293 -0.220208" rpy="0 0 0"/>
     <geometry>
       <mesh filename="package://jamie_description/meshes/head_connector_link_1.stl" scale="0.001 0.001 0.001"/>
@@ -258,5 +258,5 @@
   </visual>
   <collision>
-    <origin xyz="-0.000627 -0.035338 -0.759679" rpy="0 0 0"/>
+    <origin xyz="0.011061 0.01293 -0.220208" rpy="0 0 0"/>
     <geometry>
       <mesh filename="package://jamie_description/meshes/head_connector_link_1.stl" scale="0.001 0.001 0.001"/>
@@ -266,10 +266,10 @@
 <link name="right_shoulder_servo_v1_1">
   <inertial>
-    <origin xyz="-0.008128374894312111 -0.024681441098353595 -0.004499277410236924" rpy="0 0 0"/>
+    <origin xyz="-0.00812860742899671 -0.02468076372691968 -0.004498749573111471" rpy="0 0 0"/>
     <mass value="0.2572190211102965"/>
     <inertia ixx="4.3e-05" iyy="4.5e-05" izz="7.2e-05" ixy="2e-06" iyz="-0.0" ixz="-0.0"/>
   </inertial>
   <visual>
-    <origin xyz="-0.069825 -0.041568 -0.678692" rpy="0 0 0"/>
+    <origin xyz="-0.058137 0.006701 -0.13922" rpy="0 0 0"/>
     <geometry>
       <mesh filename="package://jamie_description/meshes/right_shoulder_servo_v1_1.stl" scale="0.001 0.001 0.001"/>
@@ -278,5 +278,5 @@
   </visual>
   <collision>
-    <origin xyz="-0.069825 -0.041568 -0.678692" rpy="0 0 0"/>
+    <origin xyz="-0.058137 0.006701 -0.13922" rpy="0 0 0"/>
     <geometry>
       <mesh filename="package://jamie_description/meshes/right_shoulder_servo_v1_1.stl" scale="0.001 0.001 0.001"/>
@@ -286,10 +286,10 @@
 <link name="right_shoulder_connector_link_1">
   <inertial>
-    <origin xyz="0.005752356597002614 0.009619046457646442 0.0024323035384365976" rpy="0 0 0"/>
+    <origin xyz="0.005752124062318106 0.009618723829080245 0.002431831375562188" rpy="0 0 0"/>
     <mass value="0.08077297877855137"/>
     <inertia ixx="3.5e-05" iyy="1.8e-05" izz="3.8e-05" ixy="0.0" iyz="-1e-06" ixz="1e-06"/>
   </inertial>
   <visual>
-    <origin xyz="-0.085625 -0.007134 -0.67419" rpy="0 0 0"/>
+    <origin xyz="-0.073937 0.041134 -0.134719" rpy="0 0 0"/>
     <geometry>
       <mesh filename="package://jamie_description/meshes/right_shoulder_connector_link_1.stl" scale="0.001 0.001 0.001"/>
@@ -298,5 +298,5 @@
   </visual>
   <collision>
-    <origin xyz="-0.085625 -0.007134 -0.67419" rpy="0 0 0"/>
+    <origin xyz="-0.073937 0.041134 -0.134719" rpy="0 0 0"/>
     <geometry>
       <mesh filename="package://jamie_description/meshes/right_shoulder_connector_link_1.stl" scale="0.001 0.001 0.001"/>
@@ -306,10 +306,10 @@
 <link name="upper_right_arm_servo_1">
   <inertial>
-    <origin xyz="-2.278268546790363e-06 0.011733258675074243 -0.025301069113281227" rpy="0 0 0"/>
+    <origin xyz="-2.510803230840186e-06 0.011732936046508276 -0.02530054127615601" rpy="0 0 0"/>
     <mass value="0.2572190211102965"/>
     <inertia ixx="7.2e-05" iyy="4.5e-05" izz="4.3e-05" ixy="0.0" iyz="2e-06" ixz="0.0"/>
   </inertial>
   <visual>
-    <origin xyz="-0.108709 -0.011881 -0.63732" rpy="0 0 0"/>
+    <origin xyz="-0.097021 0.036387 -0.097848" rpy="0 0 0"/>
     <geometry>
       <mesh filename="package://jamie_description/meshes/upper_right_arm_servo_1.stl" scale="0.001 0.001 0.001"/>
@@ -318,5 +318,5 @@
   </visual>
   <collision>
-    <origin xyz="-0.108709 -0.011881 -0.63732" rpy="0 0 0"/>
+    <origin xyz="-0.097021 0.036387 -0.097848" rpy="0 0 0"/>
     <geometry>
       <mesh filename="package://jamie_description/meshes/upper_right_arm_servo_1.stl" scale="0.001 0.001 0.001"/>
@@ -326,10 +326,10 @@
 <link name="right_upper_arm_link_1">
   <inertial>
-    <origin xyz="-0.004123117619453984 -0.017587029401361812 -0.026551245795806033" rpy="0 0 0"/>
+    <origin xyz="-0.004123350154138353 -0.017587352029927915 -0.02655071795868074" rpy="0 0 0"/>
     <mass value="0.255754845328822"/>
     <inertia ixx="0.000327" iyy="0.000305" izz="0.000135" ixy="-0.0" iyz="-1.2e-05" ixz="1e-06"/>
   </inertial>
   <visual>
-    <origin xyz="-0.113208 -0.047597 -0.622022" rpy="0 0 0"/>
+    <origin xyz="-0.10152 0.000671 -0.08255" rpy="0 0 0"/>
     <geometry>
       <mesh filename="package://jamie_description/meshes/right_upper_arm_link_1.stl" scale="0.001 0.001 0.001"/>
@@ -338,5 +338,5 @@
   </visual>
   <collision>
-    <origin xyz="-0.113208 -0.047597 -0.622022" rpy="0 0 0"/>
+    <origin xyz="-0.10152 0.000671 -0.08255" rpy="0 0 0"/>
     <geometry>
       <mesh filename="package://jamie_description/meshes/right_upper_arm_link_1.stl" scale="0.001 0.001 0.001"/>
@@ -346,10 +346,10 @@
 <link name="right_forearm_servo_1">
   <inertial>
-    <origin xyz="-0.010377890579971877 0.006384262290033325 -0.02426148248101656" rpy="0 0 0"/>
+    <origin xyz="-0.010378123114656357 0.006383939661467209 -0.024261954643891036" rpy="0 0 0"/>
     <mass value="0.2572190211102965"/>
     <inertia ixx="4.3e-05" iyy="7.1e-05" izz="4.5e-05" ixy="-0.0" iyz="2e-06" ixz="2e-06"/>
   </inertial>
   <visual>
-    <origin xyz="-0.120123 -0.024273 -0.558818" rpy="0 0 0"/>
+    <origin xyz="-0.108435 0.023995 -0.019347" rpy="0 0 0"/>
     <geometry>
       <mesh filename="package://jamie_description/meshes/right_forearm_servo_1.stl" scale="0.001 0.001 0.001"/>
@@ -358,5 +358,5 @@
   </visual>
   <collision>
-    <origin xyz="-0.120123 -0.024273 -0.558818" rpy="0 0 0"/>
+    <origin xyz="-0.108435 0.023995 -0.019347" rpy="0 0 0"/>
     <geometry>
       <mesh filename="package://jamie_description/meshes/right_forearm_servo_1.stl" scale="0.001 0.001 0.001"/>
@@ -366,10 +366,10 @@
 <link name="forearm_right_v1_1">
   <inertial>
-    <origin xyz="-0.019393772594857486 -0.006187196437031046 -0.04912306430079594" rpy="0 0 0"/>
+    <origin xyz="-0.019394005129541883 -0.006187519065597221 -0.04912253646367075" rpy="0 0 0"/>
     <mass value="0.17753961220642203"/>
     <inertia ixx="0.000376" iyy="0.000381" izz="7.2e-05" ixy="-8e-06" iyz="6.1e-05" ixz="3.4e-05"/>
   </inertial>
   <visual>
-    <origin xyz="-0.133673 -0.03141 -0.524834" rpy="0 0 0"/>
+    <origin xyz="-0.121985 0.016858 0.014638" rpy="0 0 0"/>
     <geometry>
       <mesh filename="package://jamie_description/meshes/forearm_right_v1_1.stl" scale="0.001 0.001 0.001"/>
@@ -378,5 +378,5 @@
   </visual>
   <collision>
-    <origin xyz="-0.133673 -0.03141 -0.524834" rpy="0 0 0"/>
+    <origin xyz="-0.121985 0.016858 0.014638" rpy="0 0 0"/>
     <geometry>
       <mesh filename="package://jamie_description/meshes/forearm_right_v1_1.stl" scale="0.001 0.001 0.001"/>
@@ -386,10 +386,10 @@
 <link name="left_shoulder_servo_1">
   <inertial>
-    <origin xyz="0.008128625305570812 0.023799042060737886 0.004748468071744338" rpy="0 0 0"/>
+    <origin xyz="0.008128392770885493 0.023799719432171376 0.00474899590886993" rpy="0 0 0"/>
     <mass value="0.2572190211102965"/>
     <inertia ixx="4.3e-05" iyy="4.5e-05" izz="7.2e-05" ixy="-2e-06" iyz="0.0" ixz="-0.0"/>
   </inertial>
   <visual>
-    <origin xyz="0.067625 0.006684 -0.668792" rpy="0 0 0"/>
+    <origin xyz="0.079313 0.054953 -0.12932" rpy="0 0 0"/>
     <geometry>
       <mesh filename="package://jamie_description/meshes/left_shoulder_servo_1.stl" scale="0.001 0.001 0.001"/>
@@ -398,5 +398,5 @@
   </visual>
   <collision>
-    <origin xyz="0.067625 0.006684 -0.668792" rpy="0 0 0"/>
+    <origin xyz="0.079313 0.054953 -0.12932" rpy="0 0 0"/>
     <geometry>
       <mesh filename="package://jamie_description/meshes/left_shoulder_servo_1.stl" scale="0.001 0.001 0.001"/>
@@ -406,10 +406,10 @@
 <link name="left_shoulder_connector_link_1">
   <inertial>
-    <origin xyz="-0.005752909215844815 0.009742918463123843 0.001873897803275404" rpy="0 0 0"/>
+    <origin xyz="-0.005753141750530072 0.009742595834557 0.0018734256404009109" rpy="0 0 0"/>
     <mass value="0.08076633902558729"/>
     <inertia ixx="3.5e-05" iyy="1.8e-05" izz="3.8e-05" ixy="-0.0" iyz="-0.0" ixz="-1e-06"/>
   </inertial>
   <visual>
-    <origin xyz="0.083425 -0.007363 -0.673543" rpy="0 0 0"/>
+    <origin xyz="0.095113 0.040905 -0.134072" rpy="0 0 0"/>
     <geometry>
       <mesh filename="package://jamie_description/meshes/left_shoulder_connector_link_1.stl" scale="0.001 0.001 0.001"/>
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
Commit message: added cmd_joint_state_pub

File: src/jamie_description/urdf/jamie.xacro (robot description, xacro)
@@ -5,9 +5,9 @@
 <xacro:include filename="$(find jamie_description)/urdf/jamie.gazebo" />
 <link name="base_link">
-  <inertial>
+  <!-- <inertial>
     <origin xyz="-0.011688232223622823 -0.04997378243790669 -0.12088695327313781" rpy="0 0 0"/>
     <mass value="0.8307183918921939"/>
     <inertia ixx="0.000743" iyy="0.00316" izz="0.00283" ixy="0.0" iyz="3.2e-05" ixz="-0.0"/>
-  </inertial>
+  </inertial> -->
   <visual>
     <origin xyz="0 0 0" rpy="0 0 0"/>

Commit message: Jamie Description Update

File: src/jamie_description/urdf/jamie.xacro (robot description, xacro)
@@ -5,9 +5,9 @@
 <xacro:include filename="$(find jamie_description)/urdf/jamie.gazebo" />
 <link name="base_link">
-  <!-- <inertial>
+  <inertial>
     <origin xyz="-0.011688232223622823 -0.04997378243790669 -0.12088695327313781" rpy="0 0 0"/>
     <mass value="0.8307183918921939"/>
     <inertia ixx="0.000743" iyy="0.00316" izz="0.00283" ixy="0.0" iyz="3.2e-05" ixz="-0.0"/>
-  </inertial> -->
+  </inertial>
   <visual>
     <origin xyz="0 0 0" rpy="0 0 0"/>
@@ -661,4 +661,24 @@
     <geometry>
       <mesh filename="package://jamie_description/meshes/right_foot_link_1.stl" scale="0.001 0.001 0.001"/>
+    </geometry>
+  </collision>
+</link>
+<link name="right_hand_1">
+  <inertial>
+    <origin xyz="-0.08648482679225791 -0.12490687861747213 -0.133081495861343" rpy="0 0 0"/>
+    <mass value="0.06220245659592166"/>
+    <inertia ixx="4e-06" iyy="4e-06" izz="5e-06" ixy="-0.0" iyz="-0.0" ixz="-0.0"/>
+  </inertial>
+  <visual>
+    <origin xyz="-0.19647 -0.116899 0.009254" rpy="0 0 0"/>
+    <geometry>
+      <mesh filename="package://jamie_description/meshes/right_hand_1.stl" scale="0.001 0.001 0.001"/>
+    </geometry>
+    <material name="silver"/>
+  </visual>
+  <collision>
+    <origin xyz="-0.19647 -0.116899 0.009254" rpy="0 0 0"/>
+    <geometry>
+      <mesh filename="package://jamie_description/meshes/right_hand_1.stl" scale="0.001 0.001 0.001"/>
     </geometry>
   </collision>
@@ -862,3 +882,8 @@
   <limit upper="0.785398" lower="-0.523599" effort="100" velocity="100"/>
 </joint>
+<joint name="Rigid 95" type="fixed">
+  <origin xyz="0.074485 0.133757 0.005384" rpy="0 0 0"/>
+  <parent link="forearm_right_v1_1"/>
+  <child link="right_hand_1"/>
+</joint>
 </robot>
